Commit message: velocity splitter

File: src/oarbot_description/urdf/base/oarbot_base.urdf.xacro (robot description, xacro)
@@ -53,5 +53,5 @@
         <box size="0.15 0.15 0.5"/>
       </geometry>
-      <origin rpy="0 0 0" xyz="0 0 -0.15"/>
+      <origin rpy="0 0 0" xyz="0 0 -0.25"/>
       <material name="white"/>
     </visual>
@@ -76,5 +76,5 @@
     <axis xyz="0 0 1"/>
     <limit effort="1000.0" lower="0" upper="0.3" velocity="0.3"/>
-    <origin xyz="0.3 0 0.3"/>
+    <origin xyz="0.3 0 0.4"/>
   </joint>
   <transmission name="support_transmission">

Commit message: vel splitter using qp

File: src/oarbot_description/urdf/base/oarbot_base.urdf.xacro (robot description, xacro)
@@ -59,4 +59,5 @@
       <geometry>
         <box size="0.15 0.15 0.3"/>
+        <origin rpy="0 0 0" xyz="0 0 -0.15"/>
       </geometry>
     </collision>
