Commit message: debug

File: src/assistive_launch/urdf/oarbot_blue_j2n6s300_standalone.xacro (robot description, xacro)
@@ -26,4 +26,5 @@
   </joint>
   <xacro:property name="robot_root" value="$(arg robot_root_name)" />
-  <xacro:j2n6s300  base_parent="${robot_root}" prefix="${robot_prefix}"/>
+  <xacro:property name="prefix" value="$(arg robot_prefix)" />
+  <xacro:j2n6s300  base_parent="${robot_root}" prefix="${prefix}"/>
 </robot>

Commit message: Adjust poses btw world frame and kinova arm roots

File: src/assistive_launch/urdf/oarbot_blue_j2n6s300_standalone.xacro (robot description, xacro)
@@ -23,5 +23,5 @@
     <child link="$(arg robot_root_name)" />
     <parent link="world" />
-    <origin xyz="0 0 0" rpy="0 0 0" />
+    <origin xyz="0 -0.5 0" rpy="0 0 0" />
   </joint>
   <xacro:property name="robot_root" value="$(arg robot_root_name)" />

File: src/assistive_launch/urdf/oarbot_silver_j2n6s300_standalone.xacro (robot description, xacro)
@@ -23,5 +23,5 @@
     <child link="$(arg robot_root_name)" />
     <parent link="world" />
-    <origin xyz="0 0 0" rpy="0 0 0" />
+    <origin xyz="0 0.5 0" rpy="0 0 3.14159265359" />
   </joint>
   <xacro:property name="robot_root" value="$(arg robot_root_name)" />

Commit message: add rviz config for both of the arms

File: src/assistive_launch/urdf/oarbot_blue_j2n6s300_standalone.xacro (robot description, xacro)
@@ -23,5 +23,5 @@
     <child link="$(arg robot_root_name)" />
     <parent link="world" />
-    <origin xyz="0 -0.5 0" rpy="0 0 0" />
+    <origin xyz="0 -0.5125 0" rpy="0 0 0" />
   </joint>
   <xacro:property name="robot_root" value="$(arg robot_root_name)" />

File: src/assistive_launch/urdf/oarbot_silver_j2n6s300_standalone.xacro (robot description, xacro)
@@ -23,5 +23,5 @@
     <child link="$(arg robot_root_name)" />
     <parent link="world" />
-    <origin xyz="0 0.5 0" rpy="0 0 3.14159265359" />
+    <origin xyz="0 0.5125 0" rpy="0 0 3.14159265359" />
   </joint>
   <xacro:property name="robot_root" value="$(arg robot_root_name)" />

Commit message: Implement mobile base to arm base tf broadcaster

File: src/assistive_launch/urdf/oarbot_blue_j2n6s300_standalone.xacro (robot description, xacro)
@@ -19,10 +19,10 @@
   <link name="$(arg robot_root_name)"/>
   <!-- for gazebo -->
-  <link name="world"/>
+  <!-- <link name="world"/>
   <joint name="connect_root_and_world" type="fixed">
     <child link="$(arg robot_root_name)" />
     <parent link="world" />
     <origin xyz="0 -0.5125 0" rpy="0 0 0" />
-  </joint>
+  </joint>  -->
   <xacro:property name="robot_root" value="$(arg robot_root_name)" />
   <xacro:property name="prefix" value="$(arg robot_prefix)" />

File: src/assistive_launch/urdf/oarbot_silver_j2n6s300_standalone.xacro (robot description, xacro)
@@ -19,10 +19,10 @@
   <link name="$(arg robot_root_name)"/>
   <!-- for gazebo -->
-  <link name="world"/>
+  <!-- <link name="world"/>
   <joint name="connect_root_and_world" type="fixed">
     <child link="$(arg robot_root_name)" />
     <parent link="world" />
     <origin xyz="0 0.5125 0" rpy="0 0 3.14159265359" />
-  </joint>
+  </joint>  -->
   <xacro:property name="robot_root" value="$(arg robot_root_name)" />
   <xacro:property name="prefix" value="$(arg robot_prefix)" />
