Commit message: debug

File: src/oarbot_description/urdf/wheels/omni_wheel.urdf.xacro (robot description, xacro)
@@ -7,7 +7,7 @@
   <xacro:property name="wheel_mass" value="6.5" /> <!-- in kg-->
   <xacro:macro name="cylinder_inertial" params="m r h">
-    <inertia  ixx="${m*(3*r*r+h*h)/12}" ixy = "0" ixz = "0"
-              iyy="${m*r*r/2}" iyz = "0"
-              izz="${m*(3*r*r+h*h)/12}" />
+    <inertia  ixx="${m*(3*r*r+h*h)/12.0}" ixy = "0" ixz = "0"
+              iyy="${m*r*r/2.0}" iyz = "0"
+              izz="${m*(3*r*r+h*h)/12.0}" />
   </xacro:macro>
   <xacro:macro name="omni_wheel" params="prefix parent *origin reflect">
@@ -17,5 +17,5 @@
       <xacro:insert_block name="origin" />
       <axis xyz="0 1 0" rpy="0 0 0" />
-      <limit effort="100" velocity="100"/>
+      <limit effort="100.0" velocity="100.0"/>
       <joint_properties damping="0.0" friction="0.0"/>
     </joint>
@@ -43,7 +43,10 @@
         <mass value="${wheel_mass}" />
         <origin xyz="0 0 0" />
-        <inertia  ixx="${wheel_mass}*(3*${wheel_radius}*${wheel_radius}+${wheel_height}*${wheel_height})/12" ixy = "0" ixz = "0"
-              iyy="${wheel_mass}*${wheel_radius}*${wheel_radius}/2" iyz = "0"
-              izz="${wheel_mass}*(3*${wheel_radius}*${wheel_radius}+${wheel_height}*${wheel_height})/12" />
+        <inertia  ixx="${wheel_mass *(3.0* wheel_radius * wheel_radius + wheel_height * wheel_height )/12.0 }" ixy = "0.0" ixz = "0.0"
+                  iyy="${wheel_mass * wheel_radius * wheel_radius /2.0 }" iyz = "0.0"
+                  izz="${wheel_mass *(3.0* wheel_radius * wheel_radius + wheel_height * wheel_height )/12.0 }" />
+        <!-- <inertia  ixx="0.0303095" ixy = "0.0" ixz = "0.0"
+                  iyy="0.05241925" iyz = "0.0"
+                  izz="0.0303095" /> -->
       </inertial>
     </link>
