Commit message: debug stl files and update dingo xacro

File: src/dingo_customization/urdf/dingo-o-prefixed.urdf.xacro (robot description, xacro)
@@ -198,5 +198,5 @@
             <mesh filename="package://dingo_customization/meshes/pvc_riser.STL"/>
         </geometry>
-        <!-- <material name="white" /> -->
+        <material name="light_grey" />
       </visual>
       <collision>
@@ -240,5 +240,5 @@
             <mesh filename="package://dingo_customization/meshes/pvc_riser_aruco_mount.STL"/>
         </geometry>
-        <!-- <material name="white" /> -->
+        <material name="light_grey" />
       </visual>
       <collision>
@@ -274,5 +274,5 @@
             <mesh filename="package://dingo_customization/meshes/pvc_riser_uwb_mount.STL"/>
         </geometry>
-        <!-- <material name="white" /> -->
+        <material name="light_grey" />
       </visual>
       <collision>

Commit message: update dingo xacrio

File: src/dingo_customization/urdf/dingo-o-prefixed.urdf.xacro (robot description, xacro)
@@ -20,6 +20,7 @@
   <xacro:property name="dummy_inertia" value="1e-09"/>
   <material name="white"><color rgba="1.0 1.0 1.0 1.0" /></material>
+  <material name="white_acrylic"><color rgba="1.0 1.0 1.0 0.1" /></material>
   <material name="dark_grey"><color rgba="0.2 0.2 0.2 1.0" /></material>
-  <material name="light_grey"><color rgba="0.4 0.4 0.4 1.0" /></material>
+  <material name="light_grey"><color rgba="0.7 0.7 0.7 1.0" /></material>
   <material name="yellow"><color rgba="0.8 0.8 0.0 1.0" /></material>
   <material name="black"><color rgba="0.15 0.15 0.15 1.0" /></material>
@@ -182,9 +183,11 @@
   <!-- Right uwb tag -->
   <xacro:uwb_tag tag_num="1" robot_prefix="${robot_prefix}">
-    <origin xyz="$(optenv DINGO_UWB_TAG_1_OFFSET 0 -0.22 0.1)" rpy="0 0 0"/>
+    <!-- <origin xyz="$(optenv DINGO_UWB_TAG_1_OFFSET 0 -0.22 0.1)" rpy="0 0 0"/> -->
+    <origin xyz="$(optenv DINGO_UWB_TAG_1_OFFSET 0 -0.22 0.1)" rpy="${PI/2} ${PI/2} 0"/>
   </xacro:uwb_tag>
   <!-- Left uwb tag -->
   <xacro:uwb_tag tag_num="2" robot_prefix="${robot_prefix}">
-    <origin xyz="$(optenv DINGO_UWB_TAG_2_OFFSET 0 0.22 0.1)" rpy="0 0 ${PI}"/>
+    <!-- <origin xyz="$(optenv DINGO_UWB_TAG_2_OFFSET 0 0.22 0.1)" rpy="0 0 ${PI}"/> -->
+    <origin xyz="$(optenv DINGO_UWB_TAG_2_OFFSET 0 0.22 0.1)" rpy="${-PI/2} ${-PI/2} 0"/>
   </xacro:uwb_tag>
   <!-- ++++++++++++++++++++++++++++++++++++++++++++++++++++++++ -->
@@ -194,5 +197,5 @@
     <link name="${robot_prefix}robot_arm_riser_link">
       <visual>
-        <origin xyz="0 0 0" rpy="0 0 0"/>
+        <origin xyz="0 0 0.003175" rpy="0 0 0"/>
         <geometry>
             <mesh filename="package://dingo_customization/meshes/pvc_riser.STL"/>
@@ -240,5 +243,5 @@
             <mesh filename="package://dingo_customization/meshes/pvc_riser_aruco_mount.STL"/>
         </geometry>
-        <material name="light_grey" />
+        <material name="white_acrylic" />
       </visual>
       <collision>

Commit message: debug

File: src/dingo_customization/urdf/dingo-o-prefixed.urdf.xacro (robot description, xacro)
@@ -184,5 +184,5 @@
   <xacro:uwb_tag tag_num="1" robot_prefix="${robot_prefix}">
     <!-- <origin xyz="$(optenv DINGO_UWB_TAG_1_OFFSET 0 -0.22 0.1)" rpy="0 0 0"/> -->
-    <origin xyz="$(optenv DINGO_UWB_TAG_1_OFFSET 0 -0.22 0.1)" rpy="${PI/2} ${PI/2} 0"/>
+    <origin xyz="$(optenv DINGO_UWB_TAG_1_OFFSET 0 -0.22 0.1)" rpy="${PI/2} ${-PI/2} 0"/>
   </xacro:uwb_tag>
   <!-- Left uwb tag -->
@@ -243,5 +243,5 @@
             <mesh filename="package://dingo_customization/meshes/pvc_riser_aruco_mount.STL"/>
         </geometry>
-        <material name="white_acrylic" />
+        <material name="light_grey" />
       </visual>
       <collision>
@@ -277,5 +277,5 @@
             <mesh filename="package://dingo_customization/meshes/pvc_riser_uwb_mount.STL"/>
         </geometry>
-        <material name="light_grey" />
+        <material name="white_acrylic" />
       </visual>
       <collision>

Commit message: debug

File: src/dingo_customization/urdf/dingo-o-prefixed.urdf.xacro (robot description, xacro)
@@ -20,7 +20,7 @@
   <xacro:property name="dummy_inertia" value="1e-09"/>
   <material name="white"><color rgba="1.0 1.0 1.0 1.0" /></material>
-  <material name="white_acrylic"><color rgba="1.0 1.0 1.0 0.1" /></material>
   <material name="dark_grey"><color rgba="0.2 0.2 0.2 1.0" /></material>
   <material name="light_grey"><color rgba="0.7 0.7 0.7 1.0" /></material>
+  <material name="light_grey_acyrlic"><color rgba="0.7 0.7 0.7 0.5" /></material>
   <material name="yellow"><color rgba="0.8 0.8 0.0 1.0" /></material>
   <material name="black"><color rgba="0.15 0.15 0.15 1.0" /></material>
@@ -277,5 +277,5 @@
             <mesh filename="package://dingo_customization/meshes/pvc_riser_uwb_mount.STL"/>
         </geometry>
-        <material name="white_acrylic" />
+        <material name="light_grey_acyrlic" />
       </visual>
       <collision>

Commit message: Create a launch file that sets robot description parameters to be able to visualize the robot models in RVIZ during a rosbag playback

File: src/dingo_customization/urdf/dingo-o-prefixed.urdf.xacro (robot description, xacro)
@@ -184,10 +184,12 @@
   <xacro:uwb_tag tag_num="1" robot_prefix="${robot_prefix}">
     <!-- <origin xyz="$(optenv DINGO_UWB_TAG_1_OFFSET 0 -0.22 0.1)" rpy="0 0 0"/> -->
-    <origin xyz="$(optenv DINGO_UWB_TAG_1_OFFSET 0 -0.22 0.1)" rpy="${PI/2} ${-PI/2} 0"/>
+    <!-- <origin xyz="$(optenv DINGO_UWB_TAG_1_OFFSET 0 -0.22 0.1)" rpy="${PI/2} ${-PI/2} 0"/> -->
+    <origin xyz="$(optenv DINGO_UWB_TAG_1_OFFSET 0.177 -0.24 0.543175)" rpy="${PI/2} ${-PI/2} 0"/>
   </xacro:uwb_tag>
   <!-- Left uwb tag -->
   <xacro:uwb_tag tag_num="2" robot_prefix="${robot_prefix}">
     <!-- <origin xyz="$(optenv DINGO_UWB_TAG_2_OFFSET 0 0.22 0.1)" rpy="0 0 ${PI}"/> -->
-    <origin xyz="$(optenv DINGO_UWB_TAG_2_OFFSET 0 0.22 0.1)" rpy="${-PI/2} ${-PI/2} 0"/>
+    <!-- <origin xyz="$(optenv DINGO_UWB_TAG_2_OFFSET 0 0.22 0.1)" rpy="${-PI/2} ${-PI/2} 0"/> -->
+    <origin xyz="$(optenv DINGO_UWB_TAG_2_OFFSET 0.143 0.24 0.543175)" rpy="${-PI/2} ${-PI/2} 0"/>
   </xacro:uwb_tag>
   <!-- ++++++++++++++++++++++++++++++++++++++++++++++++++++++++ -->
